Commit message: KScale Biped Configuration Updates
Problem
=======
1. Tree Tracking KScale related files in `exts/bipedal_locomotion`
   instead of `environments`
2. Actuator Pose and Nominal Joint Pose needs tuning for easier learning
   of efficient and stable gait
3. KScale Biped X axis facing sidewards in URDF which is imcompatible
   with IsaacLab
4. Need to implement and integrate symmetry data augmentation for KScale
   Biped
5. Need to compute and add Sole limits for KScale biped for feet
   velocity rewards
6. No rewards for penalising arbitrary hip yaw leading to duck or pigeon
   footed stance
7. Kscale Biped not integrated with evaluation scripts

Solution
========
1. Moved all files from `exts/bipedal_locomotion` to `environments` to
   ensure all KScale Biped related files are in `environments`
2. Corrected Actuator gains in
   `environments/environments/assets/config/kscale_identified_cfg.py`
   to ensure the joints stiffness and damping are set according to joint
   role
3. Rotated the root link in
   `environments/environments/assets/urdf/solefoot/kscale/kscale.urdf`
   to ensure x is facing forwards. Updated Moment of Inertia according
   to rotated root link
4. Added Symmetry Data augmentation for KScale biped in
   `environments/environments/tasks/locomotion/mdp/symmetry/kscale.py`
   and integrated into `class KscaleFlatPPORunnerCfg` in
   `environments/environments/tasks/locomotion/agents/limx_rsl_rl_ppo_cfg.py`
5. Added `KSCALE_SOLE_OFFSETS`, `rew_foot_clearance`, `pen_foot_landing`
   and `pen_feet_impact` in
   `environments/environments/tasks/locomotion/cfg/SF/kscale_base_env_cfg.py`
6. Added `pen_feet_heading` to penalise deviation between feet heading
   and base heading in
   `environments/environments/tasks/locomotion/cfg/SF/kscale_base_env_cfg.py`
7. Updated `feet_yaw_alignment` in
   `environments/environments/tasks/locomotion/mdp/rewards.py` to
   implement feet yaw alignment following Booster Gym implementation for
   the KScale Biped
8. Added robot profile selection to integrate KScale biped into
   `scripts/rsl_rl/play.py`

Note
====
1. Updated all documentation in @context/ and @plans regarding KScale
   Biped
2. Need to remove STL files from git tracking

File: environments/environments/assets/urdf/solefoot/kscale/kscale.urdf (robot description, URDF)
Before this commit: robot biped, 13 links, 12 joints
Joints:
- joint left_hip_pitch_04: origin xyz=0.055 -0.0246054 -0.0595116 rpy=1.5708 0 -1.5708 -> xyz=0.0246054 0.055 -0.0595116 rpy=1.5708 0 -3.67321e-06
- joint right_hip_pitch_04: origin xyz=-0.055 -0.0246054 -0.0595116 rpy=1.5708 0 1.5708 -> xyz=0.0246054 -0.055 -0.0595116 rpy=1.5708 0 -3.14159
